File: input_output_board/input_output_board.kicad_pcb (KiCad board)
At the start: 2 copper layers, 203.2 x 53.3 mm, 23 parts, among them J1 Neutrik_NCJ6FA-H, J2 Neutrik_NCJ6FA-H, J3 Neutrik_NCJ6FA-H, J4 Neutrik_NCJ6FA-H, J5 AudioJack3, J6 Conn_02x05_Odd_Even, J7 Molex_SL_01x04_Male, J8 Molex_SL_01x04_Male, K1 G6S-2, K2 G6S-2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

Commit message: update relay placement
Parts:
- moved D1 19.7 mm to (65.4, 57.8), turned to 270 degrees
- moved D2 19.7 mm to (104.8, 57.8), turned to 270 degrees
- moved D3 19.7 mm to (144.1, 58.4), turned to 270 degrees
- moved D5 19.7 mm to (222.9, 58.4), turned to 270 degrees
- moved D4 19.7 mm to (183.5, 58.4), turned to 270 degrees
- moved K1 5.72 mm to (52.7, 58.4), turned to 270 degrees
- moved K2 5.72 mm to (92.1, 58.4), turned to 270 degrees
- moved K3 5.72 mm to (131.4, 58.4), turned to 270 degrees
- moved K4 5.72 mm to (170.8, 58.4), turned to 270 degrees
- moved K5 5.72 mm to (210.2, 58.4), turned to 270 degrees
Other:
- outline, holes or cut-outs redrawn

Commit message: complete initial layout
Parts:
- moved J6 85.8 mm to (197.5, 70.5), turned to 90 degrees
- moved J7 62.9 mm to (114.9, 58.4)
- moved D5 15.9 mm to (215.3, 72.4), turned to 180 degrees
- moved D2 15.5 mm to (99.7, 72.4), turned to 180 degrees
- moved D1 15.5 mm to (60.3, 72.4), turned to 180 degrees
- moved D3 15.1 mm to (138.4, 72.4), turned to 180 degrees
- moved D4 15.1 mm to (177.8, 72.4), turned to 180 degrees
- moved J8 14.6 mm to (228.0, 71.1)
- moved K3 7.10 mm to (138.4, 59.7), turned to 180 degrees
- moved K4 7.10 mm to (177.8, 59.7), turned to 180 degrees
- moved K1 7.10 mm to (59.7, 59.7), turned to 180 degrees
- moved K2 7.10 mm to (99.1, 59.7), turned to 180 degrees
- moved K5 5.24 mm to (215.3, 59.7), turned to 180 degrees
Connections:
- J6 pad 1: /input1_select -> GNDD
- J6 pad 10: GNDD -> /output_mute_select
- J6 pad 2: GNDD -> /input1_select
- J6 pad 3: /input2_select -> GNDD
- J6 pad 4: GNDD -> /input2_select
- J6 pad 5: /input3_select -> GNDD
- J6 pad 6: GNDD -> /input3_select
- J6 pad 7: /input4_select -> GNDD
- J6 pad 8: GNDD -> /input4_select
- J6 pad 9: /output_mute_select -> GNDD
Routing:
- net /input1_select: track 0.00 -> 144.7 mm
- net /input_selected_hot: track 0.00 -> 124.9 mm
- net /input_selected_cold: track 0.00 -> 123.1 mm
- net /input2_select: track 0.00 -> 105.6 mm
- net GNDD: track 0.00 -> 68.9 mm, vias 0 -> 4
- net /input3_select: track 0.00 -> 67.0 mm
- net /output_cold: track 0.00 -> 37.0 mm
- net /output_mute_select: track 0.00 -> 37.0 mm
- net Net-(J5-PadT): track 0.00 -> 35.8 mm
- net Net-(J5-PadR): track 0.00 -> 29.6 mm
- net /input2_hot: track 0.00 -> 25.3 mm
- net /input4_hot: track 0.00 -> 25.3 mm
- net /input3_hot: track 0.00 -> 25.3 mm
- net /input1_hot: track 0.00 -> 25.3 mm
- net /input4_select: track 0.00 -> 21.8 mm
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- added copper zone on B.Cu, net /input_shield
- added copper zone on B.Cu, net /output_shield
- added copper zone on B.Cu, net GNDD
Other:
- outline, holes or cut-outs redrawn
- net class relay control: clearance 0.508 -> 0.3048
- board text added: "TODO align output jack with input jack make sure all output jacks are properly positioned FIX RELAY FOOTPRINTS check output jack footprint"
- board text removed: "TODO align output jack with input jack make sure all output jacks are properly positioned FIX RELAY FOOTPRINTS"

Commit message: fix DRC error and move board on page. NOTE: several items left in TODO
Parts:
- moved J5 38.1 mm to (223.5, 66.0)
- moved K1 38.1 mm to (59.7, 97.8)
- moved K2 38.1 mm to (99.1, 97.8)
- moved K3 38.1 mm to (138.4, 97.8)
- moved K4 38.1 mm to (177.8, 97.8)
- moved K5 38.1 mm to (215.3, 97.8)
- moved H1 38.1 mm to (76.2, 67.3)
- moved H2 38.1 mm to (115.6, 67.3)
- moved H3 38.1 mm to (154.9, 67.3)
- moved H4 38.1 mm to (194.3, 67.3)
- moved H5 38.1 mm to (231.1, 67.3)
- moved J1 38.1 mm to (49.5, 81.3)
- moved J2 38.1 mm to (88.9, 81.3)
- moved J3 38.1 mm to (128.3, 81.3)
- moved J4 38.1 mm to (167.6, 81.3)
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Routing:
- net GNDD: track 68.9 -> 70.6 mm

Commit message: update chassis grounding in input/output board because jacks connect directly to chassis
Parts:
- removed H1, H2, H3, H4, H5: MountingHole_Pad, MountingHole:MountingHole_3.2mm_M3_Pad_Via
