File: power_supply/power_supply.kicad_pcb (KiCad board)
At the start: 2 copper layers, 100 x 70 mm, 61 parts, among them J1 Conn_01x04_Male, J2 Conn_01x03_Male, J3 Conn_01x03_Male, J4 Conn_01x03_Male, J5 Conn_01x02_Male, J6 Conn_01x02_Male, U1 LM7815_TO220, U2 LM7915_TO220, U3 LM7815_TO220

Commit message: update project info on silk label
Other:
- board text added: "Power Supply rev0 Preamp 2019 G. Keeth 2019-06-09"
- board text removed: "Power Supply for Preamp 2019 rev0 G. Keeth 2019-06-09"
Changed lines of the file:
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@@
       (padsonsilk false)
       (subtractmaskfromsilk false)
-      (outputformat 4)
+      (outputformat 1)
       (mirror false)
-      (drillshape 2)
+      (drillshape 0)
       (scaleselection 1)
-      (outputdirectory "pdf"))
+      (outputdirectory "fab/"))
   )
   (net 0 "")
@@
     )
   )
-  (gr_text "Power Supply for Preamp 2019 rev0\nG. Keeth\n2019-06-09" (at 92.71 85.09) (layer B.SilkS)
+  (gr_text "Power Supply rev0\nPreamp 2019\nG. Keeth\n2019-06-09" (at 92.71 85.09) (layer B.SilkS)
     (effects (font (size 1 1) (thickness 0.15)) (justify left mirror))
   )

Commit message: update project rev to 0.1
Parts:
- R4, R5, R6: footprint Capacitor_SMD:C_0603_1608Metric_Pad1.05x0.95mm_HandSolder -> Resistor_SMD:R_0603_1608Metric_Pad1.05x0.95mm_HandSolder
Changed lines of the file:
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@@
   (title_block
     (title "Power Supply Board")
-    (date 2019-06-09)
-    (rev 0)
+    (date 2019-06-10)
+    (rev 0.1)
     (company "G. Keeth")
     (comment 1 "Preamp 2019")
@@
     (add_net "Net-(F2-Pad1)")
   )
-  (module Capacitor_SMD:C_0603_1608Metric_Pad1.05x0.95mm_HandSolder (layer F.Cu)
+  (module Resistor_SMD:R_0603_1608Metric_Pad1.05x0.95mm_HandSolder (layer F.Cu)
     (at 83.82 134.62 270)
-    (descr "Capacitor SMD 0603 (1608 Metric), square (rectangular) end terminal, IPC_7351 nominal with elongated pad for handsoldering. (Body size source: http://www.tortai-tech.com/upload/download/2011102023233369053.pdf), generated with kicad-footprint-generator")
-    (tags "capacitor handsolder")
+    (descr "Resistor SMD 0603 (1608 Metric), square (rectangular) end terminal, IPC_7351 nominal with elongated pad for handsoldering. (Body size source: http://www.tortai-tech.com/upload/download/2011102023233369053.pdf), generated with kicad-footprint-generator")
+    (tags "resistor handsolder")
     (attr smd)
-    (fp_text reference R6 (at -2.921 0 90) (layer F.SilkS)
+    (fp_text reference R6 (at 0 -1.43 90) (layer F.SilkS)
       (effects (font (size 1 1) (thickness 0.15)))
     )
@@
     (pad 1 smd roundrect (at -0.875 0 270) (size 1.05 0.95) (layers F.Cu F.Paste F.Mask) (roundrect_rratio 0.25)
       (net 18 Vrelay))
-    (model ${KISYS3DMOD}/Capacitor_SMD.3dshapes/C_0603_1608Metric.wrl
+    (model ${KISYS3DMOD}/Resistor_SMD.3dshapes/R_0603_1608Metric.wrl
       (at (xyz 0 0 0))
       (scale (xyz 1 1 1))
@@
     )
   )
-  (module Capacitor_SMD:C_0603_1608Metric_Pad1.05x0.95mm_HandSolder (layer F.Cu)
+  (module Resistor_SMD:R_0603_1608Metric_Pad1.05x0.95mm_HandSolder (layer F.Cu)
     (at 135.128 99.822)
-    (descr "Capacitor SMD 0603 (1608 Metric), square (rectangular) end terminal, IPC_7351 nominal with elongated pad for handsoldering. (Body size source: http://www.tortai-tech.com/upload/download/2011102023233369053.pdf), generated with kicad-footprint-generator")
-    (tags "capacitor handsolder")
+    (descr "Resistor SMD 0603 (1608 Metric), square (rectangular) end terminal, IPC_7351 nominal with elongated pad for handsoldering. (Body size source: http://www.tortai-tech.com/upload/download/2011102023233369053.pdf), generated with kicad-footprint-generator")
+    (tags "resistor handsolder")
     (attr smd)
-    (fp_text reference R5 (at 0 1.524) (layer F.SilkS)
+    (fp_text reference R5 (at 0 -1.43) (layer F.SilkS)
       (effects (font (size 1 1) (thickness 0.15)))
     )
@@
     (pad 1 smd roundrect (at -0.875 0) (size 1.05 0.95) (layers F.Cu F.Paste F.Mask) (roundrect_rratio 0.25)
       (net 14 GNDA))
-    (model ${KISYS3DMOD}/Capacitor_SMD.3dshapes/C_0603_1608Metric.wrl
+    (model ${KISYS3DMOD}/Resistor_SMD.3dshapes/R_0603_1608Metric.wrl
       (at (xyz 0 0 0))
       (scale (xyz 1 1 1))
@@
     )
   )
-  (module Capacitor_SMD:C_0603_1608Metric_Pad1.05x0.95mm_HandSolder (layer F.Cu)
+  (module Resistor_SMD:R_0603_1608Metric_Pad1.05x0.95mm_HandSolder (layer F.Cu)
     (at 128.27 139.7 90)
-    (descr "Capacitor SMD 0603 (1608 Metric), square (rectangular) end terminal, IPC_7351 nominal with elongated pad for handsoldering. (Body size source: http://www.tortai-tech.com/upload/download/2011102023233369053.pdf), generated with kicad-footprint-generator")
-    (tags "capacitor handsolder")
+    (descr "Resistor SMD 0603 (1608 Metric), square (rectangular) end terminal, IPC_7351 nominal with elongated pad for handsoldering. (Body size source: http://www.tortai-tech.com/upload/download/2011102023233369053.pdf), generated with kicad-footprint-generator")
+    (tags "resistor handsolder")
     (attr smd)
     (fp_text reference R4 (at 0 -1.43 90) (layer F.SilkS)
@@
     (pad 1 smd roundrect (at -0.875 0 90) (size 1.05 0.95) (layers F.Cu F.Paste F.Mask) (roundrect_rratio 0.25)
       (net 4 VCC))
-    (model ${KISYS3DMOD}/Capacitor_SMD.3dshapes/C_0603_1608Metric.wrl
+    (model ${KISYS3DMOD}/Resistor_SMD.3dshapes/R_0603_1608Metric.wrl
       (at (xyz 0 0 0))
       (scale (xyz 1 1 1))

Commit message: update title block
Other:
- board text added: "Power Supply rev0.1 Preamp 2019 G. Keeth 2019-06-09"
- board text removed: "Power Supply rev0 Preamp 2019 G. Keeth 2019-06-09"
Changed lines of the file:
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@@
   (page A)
   (title_block
-    (title "Power Supply Board")
+    (title "Power Supply")
     (date 2019-06-10)
     (rev 0.1)
@@
     )
   )
-  (gr_text "Power Supply rev0\nPreamp 2019\nG. Keeth\n2019-06-09" (at 92.71 85.09) (layer B.SilkS)
+  (gr_text "Power Supply rev0.1\nPreamp 2019\nG. Keeth\n2019-06-09" (at 92.71 85.09) (layer B.SilkS)
     (effects (font (size 1 1) (thickness 0.15)) (justify left mirror))
   )
