File: balanced_amplifier/input_amplifier.sch (KiCad schematic (older format))
At the start: 53 parts, among them U1 LM4562, U2 LM4562, U3 NE5532, U4 LM4562

Commit message: update balanced amplifier input/output/power connectors
Changed lines of the file:
@@
 Text HLabel 1200 1500 0    50   Input ~ 0
 right_in_cold
-Text HLabel 1200 3500 0    50   Input ~ 0
-right_in_ground
 Wire Wire Line
 	3600 1500 3100 1500
@@
 Wire Wire Line
 	1200 2900 1300 2900
-Wire Wire Line
-	1200 3500 1800 3500
-Connection ~ 1800 3500
 Connection ~ 6000 3500
 Wire Wire Line
@@
 Text HLabel 1200 4600 0    50   Input ~ 0
 left_in_cold
-Text HLabel 1200 6600 0    50   Input ~ 0
-left_in_ground
 Wire Wire Line
 	3600 4600 3100 4600
@@
 Wire Wire Line
 	1200 4600 1300 4600
-Wire Wire Line
-	1200 6600 1800 6600
-Connection ~ 1800 6600
 Connection ~ 6000 6600
 Wire Wire Line

Commit message: update footprint for volume/balance pots
Parts:
- RV1: footprint Potentiometer_THT_custom:Potentiometer_Bourns_91_Dual_Horizontal -> Potentiometer_THT_custom:Potentiometer_Bourns_91A2x-x28-xxx_Dual_Horizontal
Changed lines of the file:
@@
 F 0 "RV1" H 8430 1246 50  0000 R CNN
 F 1 "5k" H 8430 1155 50  0000 R CNN
-F 2 "Potentiometer_THT_custom:Potentiometer_Bourns_91_Dual_Horizontal" H 8500 1200 50  0001 C CNN
+F 2 "Potentiometer_THT_custom:Potentiometer_Bourns_91A2x-x28-xxx_Dual_Horizontal" H 8500 1200 50  0001 C CNN
 F 3 "https://www.bourns.com/docs/Product-Datasheets/91_95.pdf" H 8500 1200 50  0001 C CNN
 F 4 "Bourns" H 8500 1200 50  0001 C CNN "Manufacturer"
@@
 F 0 "RV1" H 8431 4254 50  0000 R CNN
 F 1 "5k" H 8431 4345 50  0000 R CNN
-F 2 "Potentiometer_THT_custom:Potentiometer_Bourns_91_Dual_Horizontal" H 8500 4300 50  0001 C CNN
+F 2 "Potentiometer_THT_custom:Potentiometer_Bourns_91A2x-x28-xxx_Dual_Horizontal" H 8500 4300 50  0001 C CNN
 F 3 "https://www.bourns.com/docs/Product-Datasheets/91_95.pdf" H 8500 4300 50  0001 C CNN
 F 4 "Bourns" H 8500 4300 50  0001 C CNN "Manufacturer"

Commit message: update footprint references for pots and output caps
Parts:
- RV1: footprint Potentiometer_THT_custom:Potentiometer_Bourns_91A2x-x28-xxx_Dual_Horizontal -> Potentiometer_THT_gkeeth:Potentiometer_Bourns_91A2x-x28-xxx_Dual_Horizontal
Changed lines of the file:
@@
 F 0 "RV1" H 8430 1246 50  0000 R CNN
 F 1 "5k" H 8430 1155 50  0000 R CNN
-F 2 "Potentiometer_THT_custom:Potentiometer_Bourns_91A2x-x28-xxx_Dual_Horizontal" H 8500 1200 50  0001 C CNN
+F 2 "Potentiometer_THT_gkeeth:Potentiometer_Bourns_91A2x-x28-xxx_Dual_Horizontal" H 8500 1200 50  0001 C CNN
 F 3 "https://www.bourns.com/docs/Product-Datasheets/91_95.pdf" H 8500 1200 50  0001 C CNN
 F 4 "Bourns" H 8500 1200 50  0001 C CNN "Manufacturer"
@@
 F 0 "RV1" H 8431 4254 50  0000 R CNN
 F 1 "5k" H 8431 4345 50  0000 R CNN
-F 2 "Potentiometer_THT_custom:Potentiometer_Bourns_91A2x-x28-xxx_Dual_Horizontal" H 8500 4300 50  0001 C CNN
+F 2 "Potentiometer_THT_gkeeth:Potentiometer_Bourns_91A2x-x28-xxx_Dual_Horizontal" H 8500 4300 50  0001 C CNN
 F 3 "https://www.bourns.com/docs/Product-Datasheets/91_95.pdf" H 8500 4300 50  0001 C CNN
 F 4 "Bourns" H 8500 4300 50  0001 C CNN "Manufacturer"
