File: balanced_amplifier/volume_control.sch (KiCad schematic (older format))
At the start: 57 parts, among them U5 LM4562, U6 LM4562, U7 LM4562, U8 LM4562

Commit message: update footprint for output cap to match actual part
Parts:
- C26, C33: footprint Capacitor_THT:C_Radial_D12.5mm_H25.0mm_P5.00mm -> Capacitor_THT:C_Radial_D12.5mm_H20.0mm_P5.00mm
Changed lines of the file:
@@
 EESchema Schematic File Version 4
 LIBS:balanced_amplifier-cache
-EELAYER 29 0
+EELAYER 30 0
 EELAYER END
 $Descr A 11000 8500
@@
 F 0 "C26" V 8448 900 50  0000 C CNN
 F 1 "220u" V 8539 900 50  0000 C CNN
-F 2 "Capacitor_THT:C_Radial_D12.5mm_H25.0mm_P5.00mm" H 8738 750 50  0001 C CNN
+F 2 "Capacitor_THT:C_Radial_D12.5mm_H20.0mm_P5.00mm" H 8738 750 50  0001 C CNN
 F 3 "http://nichicon-us.com/english/products/pdfs/e-uvp.pdf" H 8700 900 50  0001 C CNN
 F 4 "Nichicon" H 8700 900 50  0001 C CNN "Manufacturer"
@@
 F 0 "C33" V 8448 4200 50  0000 C CNN
 F 1 "220u" V 8539 4200 50  0000 C CNN
-F 2 "Capacitor_THT:C_Radial_D12.5mm_H25.0mm_P5.00mm" H 8738 4050 50  0001 C CNN
+F 2 "Capacitor_THT:C_Radial_D12.5mm_H20.0mm_P5.00mm" H 8738 4050 50  0001 C CNN
 F 3 "http://nichicon-us.com/english/products/pdfs/e-uvp.pdf" H 8700 4200 50  0001 C CNN
 F 4 "Nichicon" H 8700 4200 50  0001 C CNN "Manufacturer"

Commit message: update footprint references for pots and output caps
Parts:
- C27, C34: footprint Capacitor_THT:C_Radial_D12.5mm_H25.0mm_P5.00mm -> Capacitor_THT:C_Radial_D12.5mm_H20.0mm_P5.00mm
- RV2: footprint Potentiometer_THT_custom:Potentiometer_Bourns_91A2x-x28-xxx_Dual_Horizontal -> Potentiometer_THT_gkeeth:Potentiometer_Bourns_91A2x-x28-xxx_Dual_Horizontal
Changed lines of the file:
@@
 F 0 "RV2" H 2630 946 50  0000 R CNN
 F 1 "5k" H 2630 855 50  0000 R CNN
-F 2 "Potentiometer_THT_custom:Potentiometer_Bourns_91A2x-x28-xxx_Dual_Horizontal" H 2700 900 50  0001 C CNN
+F 2 "Potentiometer_THT_gkeeth:Potentiometer_Bourns_91A2x-x28-xxx_Dual_Horizontal" H 2700 900 50  0001 C CNN
 F 3 "https://www.bourns.com/docs/Product-Datasheets/91_95.pdf" H 2700 900 50  0001 C CNN
 F 4 "Bourns" H 2700 900 50  0001 C CNN "Manufacturer"
@@
 F 0 "RV2" H 2630 4246 50  0000 R CNN
 F 1 "5k" H 2630 4155 50  0000 R CNN
-F 2 "Potentiometer_THT_custom:Potentiometer_Bourns_91A2x-x28-xxx_Dual_Horizontal" H 2700 4200 50  0001 C CNN
+F 2 "Potentiometer_THT_gkeeth:Potentiometer_Bourns_91A2x-x28-xxx_Dual_Horizontal" H 2700 4200 50  0001 C CNN
 F 3 "https://www.bourns.com/docs/Product-Datasheets/91_95.pdf" H 2700 4200 50  0001 C CNN
 F 4 "Bourns" H 2700 4200 50  0001 C CNN "Manufacturer"
@@
 F 0 "C27" V 8348 2400 50  0000 C CNN
 F 1 "220u" V 8439 2400 50  0000 C CNN
-F 2 "Capacitor_THT:C_Radial_D12.5mm_H25.0mm_P5.00mm" H 8638 2250 50  0001 C CNN
+F 2 "Capacitor_THT:C_Radial_D12.5mm_H20.0mm_P5.00mm" H 8638 2250 50  0001 C CNN
 F 3 "http://nichicon-us.com/english/products/pdfs/e-uvp.pdf" H 8600 2400 50  0001 C CNN
 F 4 "Nichicon" H 8600 2400 50  0001 C CNN "Manufacturer"
@@
 F 0 "C34" V 8348 5700 50  0000 C CNN
 F 1 "220u" V 8439 5700 50  0000 C CNN
-F 2 "Capacitor_THT:C_Radial_D12.5mm_H25.0mm_P5.00mm" H 8638 5550 50  0001 C CNN
+F 2 "Capacitor_THT:C_Radial_D12.5mm_H20.0mm_P5.00mm" H 8638 5550 50  0001 C CNN
 F 3 "http://nichicon-us.com/english/products/pdfs/e-uvp.pdf" H 8600 5700 50  0001 C CNN
 F 4 "Nichicon" H 8600 5700 50  0001 C CNN "Manufacturer"
